File: ICE40_Board.kicad_sch (KiCad schematic)
At the start: 40 parts, among them J1 SPI, J2 EXPANSION, J3 R_HDR, J4 L_HDR, U1 AZ1117-1.2, U2 AMS1117-3.3, U3 USB4110-GF-A, U4 iCE40HX1K-VQ100, U5 FT2232HQ, U6 93LCxxC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

Commit message: added led
Parts:
- added D10: LED, LED_SMD:LED_0603_1608Metric, symbol Device:LED
- added R9: 330R, Resistor_SMD:R_0603_1608Metric, symbol Device:R
Connections:
- net +5V: now also R9.2
- net GND: now also D10.1 (K)
- new net: D10.2 (A), R9.1
Changed lines of the file:
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@@
     (stroke (width 0) (type default) (color 0 0 0 0))
   )
+  (wire (pts (xy 311.15 220.98) (xy 311.15 222.885))
+    (stroke (width 0) (type default) (color 0 0 0 0))
+  )
   (wire (pts (xy 85.725 23.495) (xy 92.075 23.495))
     (stroke (width 0) (type default) (color 0 0 0 0))
@@
     (stroke (width 0) (type default) (color 0 0 0 0))
   )
+  (wire (pts (xy 311.15 230.505) (xy 311.15 233.045))
+    (stroke (width 0) (type default) (color 0 0 0 0))
+  )
   (wire (pts (xy 295.91 186.69) (xy 276.86 186.69))
     (stroke (width 0) (type default) (color 0 0 0 0))
@@
     (stroke (width 0) (type default) (color 0 0 0 0))
   )
+  (wire (pts (xy 311.15 240.665) (xy 311.15 243.205))
+    (stroke (width 0) (type default) (color 0 0 0 0))
+  )
   (wire (pts (xy 59.69 128.905) (xy 59.69 130.81))
     (stroke (width 0) (type default) (color 0 0 0 0))
@@
     (pin "2")
   )
+  (symbol (lib_id "power:+5V") (at 311.15 220.98 0) (unit 1)
+    (in_bom yes) (on_board yes) (fields_autoplaced)
+    (property "Reference" "#PWR050" (id 0) (at 311.15 224.79 0)
+      (effects (font (size 1.27 1.27)) hide)
+    )
+    (property "Value" "+5V" (id 1) (at 311.15 215.265 0))
+    (property "Footprint" "" (id 2) (at 311.15 220.98 0)
+      (effects (font (size 1.27 1.27)) hide)
+    )
+    (property "Datasheet" "" (id 3) (at 311.15 220.98 0)
+      (effects (font (size 1.27 1.27)) hide)
+    )
+    (pin "1")
+  )
   (symbol (lib_id "power:+1V8") (at 133.985 58.42 0) (unit 1)
     (in_bom yes) (on_board yes) (fields_autoplaced)
@@
     (pin "9")
   )
+  (symbol (lib_id "power:GND") (at 311.15 243.205 0) (unit 1)
+    (in_bom yes) (on_board yes)
+    (property "Reference" "#PWR051" (id 0) (at 311.15 249.555 0)
+      (effects (font (size 1.27 1.27)) hide)
+    )
+    (property "Value" "GND" (id 1) (at 314.325 247.65 0)
+      (effects (font (size 1.27 1.27)) (justify right))
+    )
+    (property "Footprint" "" (id 2) (at 311.15 243.205 0)
+      (effects (font (size 1.27 1.27)) hide)
+    )
+    (property "Datasheet" "" (id 3) (at 311.15 243.205 0)
+      (effects (font (size 1.27 1.27)) hide)
+    )
+    (pin "1")
+  )
   (symbol (lib_id "power:GND") (at 145.415 34.29 0) (unit 1)
     (in_bom yes) (on_board yes) (fields_autoplaced)
@@
     (pin "1")
   )
+  (symbol (lib_id "Device:R") (at 311.15 226.695 180) (unit 1)
+    (in_bom yes) (on_board yes)
+    (property "Reference" "R9" (id 0) (at 309.245 226.695 90))
+    (property "Value" "330R" (id 1) (at 311.15 226.695 90))
+    (property "Footprint" "Resistor_SMD:R_0603_1608Metric" (id 2) (at 312.928 226.695 90)
+      (effects (font (size 1.27 1.27)) hide)
+    )
+    (property "Datasheet" "~" (id 3) (at 311.15 226.695 0)
+      (effects (font (size 1.27 1.27)) hide)
+    )
+    (pin "1")
+    (pin "2")
+  )
   (symbol (lib_id "power:+5V") (at 27.305 196.215 0) (unit 1)
     (in_bom yes) (on_board yes) (fields_autoplaced)
@@
     (pin "2")
   )
+  (symbol (lib_id "Device:LED") (at 311.15 236.855 90) (unit 1)
+    (in_bom yes) (on_board yes) (fields_autoplaced)
+    (property "Reference" "D10" (id 0) (at 314.325 237.1724 90)
+      (effects (font (size 1.27 1.27)) (justify right))
+    )
+    (property "Value" "LED" (id 1) (at 314.325 239.7124 90)
+      (effects (font (size 1.27 1.27)) (justify right))
+    )
+    (property "Footprint" "LED_SMD:LED_0603_1608Metric" (id 2) (at 311.15 236.855 0)
+      (effects (font (size 1.27 1.27)) hide)
+    )
+    (property "Datasheet" "~" (id 3) (at 311.15 236.855 0)
+      (effects (font (size 1.27 1.27)) hide)
+    )
+    (pin "1")
+    (pin "2")
+  )
   (symbol (lib_id "Device:LED") (at 229.87 222.885 90) (unit 1)
     (in_bom yes) (on_board yes) (fields_autoplaced)
@@
       (reference "#PWR049") (unit 1) (value "GND") (footprint "")
     )
+    (path "/1ed11e7c-ee84-4b96-be91-72a505aedae1"
+      (reference "#PWR050") (unit 1) (value "+5V") (footprint "")
+    )
+    (path "/2153b2d3-e996-49a3-b0d7-186bceefe537"
+      (reference "#PWR051") (unit 1) (value "GND") (footprint "")
+    )
     (path "/bf86ee4e-f178-4b38-839d-c8ce62a6db22"
       (reference "C1") (unit 1) (value "100n") (footprint "Capacitor_SMD:C_0603_1608Metric")
@@
       (reference "D9") (unit 1) (value "LED") (footprint "LED_SMD:LED_0603_1608Metric")
     )
+    (path "/e1fa6f9b-2a9a-4376-893f-62c8d29c4f42"
+      (reference "D10") (unit 1) (value "LED") (footprint "LED_SMD:LED_0603_1608Metric")
+    )
     (path "/0ed67eed-157f-49b1-87fa-fc37738f8a4d"
       (reference "J1") (unit 1) (value "SPI") (footprint "Connector_PinHeader_1.27mm:PinHeader_1x08_P1.27mm_Vertical")
@@
       (reference "R8") (unit 1) (value "10k") (footprint "Resistor_SMD:R_0603_1608Metric")
     )
+    (path "/75d244f1-c8b4-4eb5-80c7-3ae94b7afbfa"
+      (reference "R9") (unit 1) (value "330R") (footprint "Resistor_SMD:R_0603_1608Metric")
+    )
     (path "/81cb6de4-3919-4208-a0ce-2091647d35cf"
